File: AVC But witn an RP2040.brd (EAGLE design)
At the start: 44.1 x 78.7 mm, 45 parts, among them J1 MICRO_USB, J10 3P_HEADER, J11 3P_HEADER, J12 3P_HEADER, J13 3P_HEADER, J14 3P_HEADER, J15 3P_HEADER, J16 3P_HEADER, J17 3P_HEADER, J18 4P_HEADER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

Commit message: Add files via upload
Connections:
- net 12V: now also Q4.3, Q5.3, Q6.3; no longer Q4.2, Q5.2, Q6.2
- net T112V: now also Q4.2; no longer Q4.3
- net T212V: now also Q5.2; no longer Q5.3
- net T312V: now also Q6.2; no longer Q6.3
Routing:
- net 12V: track 124.7 -> 140.3 mm, vias 8 -> 11
- net T112V: track 4.25 -> 9.79 mm, vias 0 -> 2
- net T312V: track 4.02 -> 9.49 mm, vias 0 -> 1
- net T212V: track 4.18 -> 7.23 mm
- net GND: track 285.2 -> 282.9 mm
- net GP12: track 42.8 -> 42.1 mm
Changed lines of the file:
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@@
 <wire x1="12.975175" y1="17.5534" x2="14.1108" y2="17.5534" width="0.1524" layer="16"/>
 <wire x1="14.1108" y1="17.5534" x2="17.8549" y2="21.2975" width="0.1524" layer="16"/>
-<wire x1="26.2649" y1="21.2975" x2="27.9074" y2="22.94" width="0.3048" layer="16"/>
 <wire x1="2.58" y1="69.85" x2="2.58" y2="62.23" width="0.3048" layer="16"/>
 <wire x1="20.285059375" y1="60.7125125" x2="21.048734375" y2="59.9488375" width="0.3048" layer="1"/>
@@
 <signal name="GP3">
 <contactref element="U1" pad="5"/>
-<wire x1="12.149" y1="38.819" x2="12.149" y2="29.779" width="0.1524" layer="16"/>
+<wire x1="12.149" y1="29.779" x2="12.149" y2="38.819" width="0.1524" layer="16"/>
 <wire x1="12.149" y1="38.819" x2="17.78" y2="44.45" width="0.1524" layer="16"/>
 <via x="17.78" y="44.45" extent="1-16" drill="0.35"/>
@@
 <wire x1="18.295096875" y1="44.965096875" x2="18.519809375" y2="44.965096875" width="0.1524" layer="1"/>
 <contactref element="Q4" pad="1"/>
-<wire x1="12.149" y1="29.779" x2="11.514" y2="29.144" width="0.3048" layer="16"/>
 <wire x1="11.514" y1="29.144" x2="11.347" y2="29.144" width="0.3048" layer="16"/>
+<wire x1="11.347" y1="29.144" x2="11.982" y2="29.779" width="0.1524" layer="16"/>
+<wire x1="11.982" y1="29.779" x2="12.149" y2="29.779" width="0.1524" layer="16"/>
 </signal>
 <signal name="GP4">
@@
 <contactref element="Q6" pad="1"/>
 <wire x1="36.83" y1="20.32" x2="36.94" y2="20.32" width="0.3048" layer="16"/>
-<wire x1="36.94" y1="20.32" x2="38.42" y2="18.84" width="0.3048" layer="16"/>
+<wire x1="36.94" y1="20.32" x2="38.42" y2="18.84" width="0.1524" layer="16"/>
 </signal>
 <signal name="GP6">
@@
 <wire x1="26.9814" y1="29.5214" x2="28.3545875" y2="29.5214" width="0.1524" layer="16"/>
 <wire x1="28.3545875" y1="29.5214" x2="29.26159375" y2="30.42840625" width="0.1524" layer="16"/>
-<wire x1="29.727603125" y1="30.894415625" x2="29.26159375" y2="30.42840625" width="0.1524" layer="16"/>
 <wire x1="29.26159375" y1="30.42840625" x2="29.26159375" y2="35.4653875" width="0.1524" layer="16"/>
 <wire x1="29.26159375" y1="35.4653875" x2="29.283103125" y2="35.486896875" width="0.1524" layer="16"/>
@@
 <signal name="T112V">
 <contactref element="T_PY1" pad="P0"/>
-<contactref element="Q4" pad="3"/>
-<wire x1="9.227" y1="28.194" x2="8.973" y2="27.94" width="0.3048" layer="16"/>
-<wire x1="8.973" y1="27.94" x2="5.08" y2="27.94" width="0.3048" layer="16"/>
+<contactref element="Q4" pad="2"/>
+<wire x1="5.08" y1="27.94" x2="6.35" y2="27.94" width="0.3048" layer="16"/>
+<wire x1="6.35" y1="27.94" x2="7.62" y2="26.67" width="0.3048" layer="16"/>
+<via x="7.62" y="26.67" extent="1-16" drill="0.35"/>
+<wire x1="7.62" y1="26.67" x2="9.5532" y2="24.7368" width="0.3048" layer="1"/>
+<wire x1="9.5532" y1="24.7368" x2="9.5532" y2="24.4891125" width="0.3048" layer="1"/>
+<via x="9.5532" y="24.4891125" extent="1-16" drill="0.35"/>
+<wire x1="9.5532" y1="24.4891125" x2="9.5532" y2="25.0408875" width="0.3048" layer="16"/>
+<wire x1="9.5532" y1="25.0408875" x2="9.477" y2="25.1170875" width="0.3048" layer="16"/>
+<wire x1="9.477" y1="25.1170875" x2="9.477" y2="25.6829125" width="0.3048" layer="16"/>
+<wire x1="9.477" y1="25.6829125" x2="9.8770875" y2="26.083" width="0.3048" layer="16"/>
+<wire x1="9.8770875" y1="26.083" x2="10.186" y2="26.083" width="0.3048" layer="16"/>
+<wire x1="10.186" y1="26.083" x2="11.347" y2="27.244" width="0.3048" layer="16"/>
 </signal>
 <signal name="T312V">
 <contactref element="T_PY3" pad="P0"/>
-<contactref element="Q6" pad="3"/>
-<wire x1="39.37" y1="12.7" x2="39.37" y2="16.72" width="0.3048" layer="16"/>
+<contactref element="Q6" pad="2"/>
+<wire x1="40.32" y1="18.84" x2="39.37" y2="19.79" width="0.3048" layer="16"/>
+<wire x1="39.37" y1="19.79" x2="39.37" y2="20.32" width="0.3048" layer="16"/>
+<via x="39.37" y="20.32" extent="1-16" drill="0.35"/>
+<wire x1="39.37" y1="20.32" x2="39.37" y2="12.7" width="0.3048" layer="1"/>
 </signal>
 <signal name="T212V">
 <contactref element="T_PY2" pad="P0"/>
-<contactref element="Q5" pad="3"/>
-<wire x1="5.461" y1="16.72" x2="5.461" y2="13.081" width="0.3048" layer="16"/>
 <wire x1="5.461" y1="13.081" x2="5.08" y2="12.7" width="0.3048" layer="16"/>
+<contactref element="Q5" pad="2"/>
+<wire x1="6.411" y1="14.031" x2="6.411" y2="18.84" width="0.3048" layer="16"/>
+<wire x1="5.08" y1="12.7" x2="6.411" y2="14.031" width="0.3048" layer="16"/>
 </signal>
 <signal name="12V">
@@
 <wire x1="6.35" y1="20.32" x2="11.43" y2="25.4" width="0.3048" layer="1"/>
 <via x="11.43" y="25.4" extent="1-16" drill="0.35"/>
-<wire x1="41.91" y1="20.47" x2="41.91" y2="22.86" width="0.3048" layer="16"/>
 <via x="41.91" y="22.86" extent="1-16" drill="0.35"/>
 <wire x1="41.91" y1="22.86" x2="41.91" y2="25.4" width="0.3048" layer="1"/>
@@
 <via x="13.97" y="25.4" extent="1-16" drill="0.35"/>
 <wire x1="13.97" y1="25.4" x2="11.43" y2="25.4" width="0.3048" layer="1"/>
-<contactref element="Q5" pad="2"/>
-<contactref element="Q4" pad="2"/>
-<contactref element="Q6" pad="2"/>
 <wire x1="6.35" y1="20.32" x2="6.411" y2="20.259" width="0.3048" layer="16"/>
-<wire x1="6.411" y1="20.259" x2="6.411" y2="18.84" width="0.3048" layer="16"/>
-<wire x1="11.43" y1="27.161" x2="11.347" y2="27.244" width="0.3048" layer="16"/>
-<wire x1="11.43" y1="25.4" x2="11.43" y2="27.161" width="0.3048" layer="16"/>
-<wire x1="40.32" y1="18.84" x2="40.32" y2="18.88" width="0.3048" layer="16"/>
-<wire x1="40.32" y1="18.88" x2="41.91" y2="20.47" width="0.3048" layer="16"/>
+<contactref element="Q6" pad="3"/>
+<contactref element="Q4" pad="3"/>
+<contactref element="Q5" pad="3"/>
+<wire x1="5.461" y1="16.72" x2="5.461" y2="19.431" width="0.3048" layer="16"/>
+<wire x1="5.461" y1="19.431" x2="6.35" y2="20.32" width="0.3048" layer="16"/>
+<wire x1="11.43" y1="25.4" x2="11.43" y2="29.1947625" width="0.3048" layer="1"/>
+<wire x1="11.43" y1="29.1947625" x2="10.6501625" y2="29.9746" width="0.3048" layer="1"/>
+<via x="10.6501625" y="29.9746" extent="1-16" drill="0.35"/>
+<wire x1="10.6501625" y1="29.9746" x2="10.6362" y2="29.9885625" width="0.3048" layer="16"/>
+<wire x1="10.6362" y1="29.9885625" x2="10.6362" y2="31.81435" width="0.3048" layer="16"/>
+<via x="10.6362" y="31.81435" extent="1-16" drill="0.35"/>
+<wire x1="10.6362" y1="31.81435" x2="8.460925" y2="29.639075" width="0.3048" layer="1"/>
+<via x="8.460925" y="29.639075" extent="1-16" drill="0.35"/>
+<wire x1="8.460925" y1="29.639075" x2="9.227" y2="28.873" width="0.3048" layer="16"/>
+<wire x1="9.227" y1="28.873" x2="9.227" y2="28.194" width="0.3048" layer="16"/>
+<wire x1="39.37" y1="16.72" x2="40.85" y2="16.72" width="0.3048" layer="16"/>
+<wire x1="40.85" y1="16.72" x2="41.91" y2="17.78" width="0.3048" layer="16"/>
+<wire x1="41.91" y1="17.78" x2="41.91" y2="22.86" width="0.3048" layer="16"/>
 </signal>
 <signal name="GP15">
@@
 <wire x1="26.86285" y1="45.59078125" x2="26.86285" y2="44.75094375" width="0.1524" layer="16"/>
 <wire x1="26.86285" y1="44.75094375" x2="26.240925" y2="44.12901875" width="0.1524" layer="16"/>
-<via x="26.67" y="31.75" extent="1-16" drill="0.35"/>
+<via x="26.416" y="32.004" extent="1-16" drill="0.35"/>
 <wire x1="26.240925" y1="35.989075" x2="24.7932" y2="34.54135" width="0.1524" layer="1"/>
-<wire x1="24.7932" y1="34.54135" x2="24.7932" y2="33.6268" width="0.1524" layer="1"/>
-<wire x1="24.7932" y1="33.6268" x2="26.67" y2="31.75" width="0.1524" layer="1"/>
+<wire x1="27.5329" y1="31.877" x2="27.6599" y2="31.75" width="0.1524" layer="16"/>
+<wire x1="24.7932" y1="34.54135" x2="24.7932" y2="34.03865" width="0.1524" layer="1"/>
+<wire x1="26.416" y1="32.41585" x2="26.416" y2="32.004" width="0.1524" layer="1"/>
+<wire x1="24.7932" y1="34.03865" x2="26.416" y2="32.41585" width="0.1524" layer="1"/>
+<wire x1="26.416" y1="32.004" x2="26.67" y2="31.75" width="0.1524" layer="16"/>
 <wire x1="26.67" y1="31.75" x2="27.6599" y2="31.75" width="0.1524" layer="16"/>
 </signal>
