File: AVC But witn an RP2040.sch (EAGLE design)
At the start: 45 parts, among them J1 MICRO_USB, J10 3P_HEADER, J11 3P_HEADER, J12 3P_HEADER, J13 3P_HEADER, J14 3P_HEADER, J15 3P_HEADER, J16 3P_HEADER, J17 3P_HEADER, J18 4P_HEADER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

Commit message: Add files via upload
Connections:
- net 12V: now also Q4.D, Q5.D, Q6.D; no longer Q4.S, Q5.S, Q6.S
- net T112V: now also Q4.S; no longer Q4.D
- net T212V: now also Q5.S; no longer Q5.D
- net T312V: now also Q6.S; no longer Q6.D
Changed lines of the file:
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@@
 </segment>
 <segment>
-<pinref part="Q4" gate="G$1" pin="D"/>
-<wire x1="288.798" y1="177.546" x2="288.798" y2="180.086" width="0.1524" layer="91"/>
-<label x="288.798" y="180.086" size="1.778" layer="95"/>
+<pinref part="Q4" gate="G$1" pin="S"/>
+<wire x1="288.798" y1="167.386" x2="288.798" y2="164.846" width="0.1524" layer="91"/>
+<label x="288.798" y="164.846" size="1.778" layer="95"/>
 </segment>
 </net>
@@
 </segment>
 <segment>
-<pinref part="Q6" gate="G$1" pin="D"/>
-<wire x1="273.558" y1="177.546" x2="273.558" y2="180.086" width="0.1524" layer="91"/>
-<label x="273.558" y="180.086" size="1.778" layer="95"/>
+<pinref part="Q6" gate="G$1" pin="S"/>
+<wire x1="273.558" y1="167.386" x2="273.558" y2="164.846" width="0.1524" layer="91"/>
+<label x="273.558" y="164.846" size="1.778" layer="95"/>
 </segment>
 </net>
@@
 </segment>
 <segment>
-<pinref part="Q5" gate="G$1" pin="D"/>
-<wire x1="304.038" y1="177.546" x2="304.038" y2="180.086" width="0.1524" layer="91"/>
-<label x="304.038" y="180.086" size="1.778" layer="95"/>
+<pinref part="Q5" gate="G$1" pin="S"/>
+<wire x1="304.038" y1="167.386" x2="304.038" y2="164.846" width="0.1524" layer="91"/>
+<label x="304.038" y="164.846" size="1.778" layer="95"/>
 </segment>
 </net>
@@
 </segment>
 <segment>
-<pinref part="Q5" gate="G$1" pin="S"/>
-<wire x1="304.038" y1="167.386" x2="304.038" y2="164.846" width="0.1524" layer="91"/>
-<label x="304.038" y="164.846" size="1.778" layer="95"/>
+<pinref part="Q6" gate="G$1" pin="D"/>
+<wire x1="273.558" y1="177.546" x2="273.558" y2="180.086" width="0.1524" layer="91"/>
+<label x="273.558" y="180.086" size="1.778" layer="95"/>
 </segment>
 <segment>
-<pinref part="Q4" gate="G$1" pin="S"/>
-<wire x1="288.798" y1="167.386" x2="288.798" y2="164.846" width="0.1524" layer="91"/>
-<label x="288.798" y="164.846" size="1.778" layer="95"/>
+<pinref part="Q4" gate="G$1" pin="D"/>
+<wire x1="288.798" y1="177.546" x2="288.798" y2="180.086" width="0.1524" layer="91"/>
+<label x="288.798" y="180.086" size="1.778" layer="95"/>
 </segment>
 <segment>
-<pinref part="Q6" gate="G$1" pin="S"/>
-<wire x1="273.558" y1="167.386" x2="273.558" y2="164.846" width="0.1524" layer="91"/>
-<label x="273.558" y="164.846" size="1.778" layer="95"/>
+<pinref part="Q5" gate="G$1" pin="D"/>
+<wire x1="304.038" y1="177.546" x2="304.038" y2="180.086" width="0.1524" layer="91"/>
+<label x="304.038" y="180.086" size="1.778" layer="95"/>
 </segment>
 </net>
